File: Entwurf1.sch (EAGLE design)
At the start: 5 parts, among them X2 DTF13-12PA

Commit message: ..
Parts:
- added BREMSLEUCHTE, LICHT_LINKS, LICHT_RECHTS: Rot, Wurth_LEDs_WL-TMRW:WL-TMRW_5MM_151054RS03000_WITHOUTSTOPPER
- added LADELEITUNG, NEBELSCHLUSSLEUCHTE, RUECKFAHRLEUCHTE, STROMVERSORGUNG: Grün, Wurth_LEDs_WL-TMRW:WL-TMRW_5MM_151054GS03000_WITHOUTSTOPPER
- added R3, R4, R5, R6, R7, R8, R9: 680, resistor:R-EU_0204/7
Connections:
- net BLINKER_LINKS renamed BLINKER_LINKS_1
- net BLINKER_RECHTS renamed BLINKER_RECHTS_4
- removed net BREMSLEUCHTE: X2G$1.6
- removed net LADELEITUNG: X2G$1.10
- removed net LICHT_LINKS: X2G$1.7
- removed net LICHT_RECHTS: X2G$1.5
- removed net MASSE: R1.1, R2.1, X2G$1.3
- removed net MASSE_9_12: X2G$1.12
- removed net MASSE_LADELEITUNG: X2G$1.11
- removed net NEBELSCHLUSSLEUCHTE: X2G$1.2
- removed net RUECKFAHRLEUCHTE: X2G$1.8
- removed net STROMVERSORGUNG: X2G$1.9
- new net BREMSLEUCHTE_6: BREMSLEUCHTE.+, X2G$1.6
- new net LADELEITUNG_10: LADELEITUNG.+, X2G$1.10
- new net LICHT_LINKS_7: LICHT_LINKS.+, X2G$1.7
- new net LICHT_RECHTS_5: LICHT_RECHTS.+, X2G$1.5
- new net MASSE_1_8: R1.1, R2.1, R3.1, R4.1, R5.1, R6.1, R9.1, X2G$1.3
- new net MASSE_9: R7.1, R8.1, X2G$1.12
- new net N$1: LICHT_LINKS.-, R3.2
- new net N$2: LICHT_RECHTS.-, R4.2
- new net N$4: BREMSLEUCHTE.-, R5.2
- new net N$6: NEBELSCHLUSSLEUCHTE.-, R6.2
- new net N$7: R7.2, STROMVERSORGUNG.-
- new net N$8: LADELEITUNG.-, R8.2
- new net N$9: R9.2, RUECKFAHRLEUCHTE.-
- new net NEBELSCHLUSSLEUCHTE_2: NEBELSCHLUSSLEUCHTE.+, X2G$1.2
- new net RUECKFAHRLEUCHTE_8: RUECKFAHRLEUCHTE.+, X2G$1.8
- new net STROMVERSORGUNG_9: STROMVERSORGUNG.+, X2G$1.9
