File: Platine_3.brd (EAGLE design)
At the start: 88.9 x 101.6 mm, 0 parts

Commit message: Done !
Routing:
- removed copper zone on layer 1, net MASSE_1_8
- removed copper zone on layer 16, net MASSE_1_8
Other:
- outline, holes or cut-outs redrawn
