File: Platine_2.brd (EAGLE design)
At the start: 88.9 x 101.6 mm, 19 parts, among them X2 DTF13-12PA

Commit message: Diode added !
Parts:
- added D1, D2: 1N4004, Diodes:DO-41
Connections:
- new net N$10: D1.C, X2.12
- new net N$11: D2.C, X2.3
- net MASSE_1_8: now also D2.A; no longer X2.3
- net MASSE_9: now also D1.A; no longer X2.12
Routing:
- net N$10: track 0.00 -> 18.2 mm
- net N$11: track 0.00 -> 4.95 mm
- net MASSE_9: track 74.3 -> 76.5 mm
Changed lines of the file:
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@@
 <drawing>
 <settings>
-<setting alwaysvectorfont="no"/>
+<setting alwaysvectorfont="yes"/>
 <setting verticaltext="up"/>
 </settings>
@@
 </layers>
 <board>
-<fusionsync huburn="a.YnVzaW5lc3M6bXNtdWM" projecturn="a.YnVzaW5lc3M6bXNtdWMjRDIwMjAwMTIwMjU2OTQxODU2" f3durn="urn:adsk.wipprod:dm.lineage:IUqRmy3CQzOHNwqusI1-PQ" pcbguid="4c452567-f71f-4f3b-8b2b-90f16c76dd37" lastpulledtime="" lastsyncedchangeguid="" latestrevisionid="2a4d4074-0cd2-4306-9f60-acfb19890fe7" lastsyncedrevisionid="2a4d4074-0cd2-4306-9f60-acfb19890fe7" lastboardhashguid="e7ef53f0-1e01-685d-f884-12b6b30a0554" lastpushedtime="2021-11-17T06:51:52Z" linktopcb3d="true"/>
+<fusionsync huburn="a.YnVzaW5lc3M6bXNtdWM" projecturn="a.YnVzaW5lc3M6bXNtdWMjRDIwMjAwMTIwMjU2OTQxODU2" f3durn="urn:adsk.wipprod:dm.lineage:IUqRmy3CQzOHNwqusI1-PQ" pcbguid="" lastpulledtime="" lastsyncedchangeguid="" latestrevisionid="4bd172e8-aa06-4833-81b5-f9206e29f622" lastsyncedrevisionid="4bd172e8-aa06-4833-81b5-f9206e29f622" lastboardhashguid="836c3ede-1ee6-a0b7-3cca-db3b111b415d" lastpushedtime="2021-11-17T12:44:38Z" linktopcb3d="true"/>
 <plain>
 <wire x1="-44.45" y1="92.25" x2="-44.45" y2="-3.35" width="0" layer="20"/>
@@
 <attribute name="VALUE" x="6.8326" y="72.0344" size="0.9906" layer="27" ratio="10" rot="R90"/>
 </element>
+<element name="D1" library="Diodes" library_urn="urn:adsk.eagle:library:11396254" package="DO-41" package3d_urn="urn:adsk.eagle:package:10898391/4" value="1N4004" x="-27.94" y="2.54" smashed="yes" rot="R180">
+<attribute name="CREATED_BY" value="PCBLayout.com" x="-27.94" y="2.54" size="1.778" layer="27" rot="R180" display="off"/>
+<attribute name="DIGIKEY_PART_NUMBER" value="1N4004MSCT-ND" x="-27.94" y="2.54" size="1.778" layer="27" rot="R180" display="off"/>
+<attribute name="MANUFACTURER" value="Micro Commercial Co" x="-27.94" y="2.54" size="1.778" layer="27" rot="R180" display="off"/>
+<attribute name="MPN" value="1N4004" x="-27.94" y="2.54" size="1.778" layer="27" rot="R180" display="off"/>
+<attribute name="NAME" x="-22.44" y="0.79" size="1.27" layer="25" ratio="10" rot="R180"/>
+<attribute name="PACKAGE" value="DO-41" x="-27.94" y="2.54" size="1.778" layer="27" rot="R180" display="off"/>
+<attribute name="VALUE" x="-22.44" y="5.54" size="1.27" layer="27" ratio="10" rot="R180"/>
+</element>
+<element name="D2" library="Diodes" library_urn="urn:adsk.eagle:library:11396254" package="DO-41" package3d_urn="urn:adsk.eagle:package:10898391/4" value="1N4004" x="-3.302" y="11.049" smashed="yes" rot="R90">
+<attribute name="CREATED_BY" value="PCBLayout.com" x="-3.302" y="11.049" size="1.778" layer="27" rot="R90" display="off"/>
+<attribute name="DIGIKEY_PART_NUMBER" value="1N4004MSCT-ND" x="-3.302" y="11.049" size="1.778" layer="27" rot="R90" display="off"/>
+<attribute name="MANUFACTURER" value="Micro Commercial Co" x="-3.302" y="11.049" size="1.778" layer="27" rot="R90" display="off"/>
+<attribute name="MPN" value="1N4004" x="-3.302" y="11.049" size="1.778" layer="27" rot="R90" display="off"/>
+<attribute name="NAME" x="-5.052" y="5.549" size="1.27" layer="25" ratio="10" rot="R90"/>
+<attribute name="PACKAGE" value="DO-41" x="-3.302" y="11.049" size="1.778" layer="27" rot="R90" display="off"/>
+<attribute name="VALUE" x="-0.302" y="5.549" size="1.27" layer="27" ratio="10" rot="R90"/>
+</element>
 </elements>
 <signals>
@@
 </signal>
 <signal name="MASSE_1_8">
-<contactref element="X2" pad="3"/>
 <contactref element="R2" pad="1"/>
 <contactref element="R1" pad="1"/>
@@
 <contactref element="R6" pad="1"/>
 <contactref element="R9" pad="1"/>
-<via x="-2.225" y="4.45" extent="1-16" drill="0.35"/>
 <via x="4.45" y="11.125" extent="1-16" drill="0.35"/>
 <via x="4.45" y="13.35" extent="1-16" drill="0.35"/>
@@
 <via x="-13.35" y="8.9" extent="1-16" drill="0.35"/>
 <via x="-13.35" y="6.675" extent="1-16" drill="0.35"/>
-<via x="-4.45" y="6.675" extent="1-16" drill="0.35"/>
 <via x="-4.45" y="8.9" extent="1-16" drill="0.35"/>
 <via x="-4.45" y="11.125" extent="1-16" drill="0.35"/>
 <via x="-2.225" y="11.125" extent="1-16" drill="0.35"/>
 <via x="-2.225" y="8.9" extent="1-16" drill="0.35"/>
-<via x="-2.225" y="6.675" extent="1-16" drill="0.35"/>
 <via x="-4.45" y="4.45" extent="1-16" drill="0.35"/>
 <via x="-4.45" y="2.225" extent="1-16" drill="0.35"/>
@@
 <via x="-15.575" y="24.475" extent="1-16" drill="0.35"/>
 <via x="-8.9" y="24.475" extent="1-16" drill="0.35"/>
+<contactref element="D2" pad="A"/>
+<via x="-20.97" y="1.595" extent="1-16" drill="0.35"/>
+<via x="-26.05" y="-3.485" extent="1-16" drill="0.35"/>
 </signal>
 <signal name="N$3">
@@
 </signal>
 <signal name="MASSE_9">
-<contactref element="X2" pad="12"/>
 <contactref element="R7" pad="1"/>
 <contactref element="R8" pad="1"/>
-<wire x1="-11.125" y1="-2.2225" x2="-8.9" y2="-4.4475" width="0.8128" layer="16"/>
 <wire x1="-8.9" y1="-4.4475" x2="-8.9" y2="-4.45" width="0.8128" layer="16"/>
 <wire x1="20.95" y1="-4.45" x2="31.75" y2="6.35" width="0.8128" layer="16"/>
 <wire x1="-8.9" y1="-4.45" x2="20.95" y2="-4.45" width="0.8128" layer="16"/>
-<wire x1="-11.125" y1="-2.2225" x2="-13.35" y2="-4.4475" width="0.8128" layer="16"/>
-<wire x1="-13.35" y1="-4.4475" x2="-13.35" y2="-4.45" width="0.8128" layer="16"/>
+<wire x1="-13.35" y1="-4.45" x2="-13.35" y2="-4.4475" width="0.8128" layer="16"/>
 <wire x1="-20.95" y1="-4.45" x2="-31.75" y2="6.35" width="0.8128" layer="16"/>
 <wire x1="-13.35" y1="-4.45" x2="-20.95" y2="-4.45" width="0.8128" layer="16"/>
+<contactref element="D1" pad="A"/>
+<wire x1="-31.75" y1="6.35" x2="-31.75" y2="3.055" width="0.8128" layer="16"/>
+<wire x1="-31.75" y1="3.055" x2="-32.265" y2="2.54" width="0.8128" layer="16"/>
+<wire x1="-13.35" y1="-4.4475" x2="-8.9025" y2="-4.4475" width="0.8128" layer="16"/>
+<wire x1="-8.9025" y1="-4.4475" x2="-8.9" y2="-4.45" width="0.8128" layer="16"/>
+</signal>
+<signal name="N$10">
+<contactref element="X2" pad="12"/>
+<contactref element="D1" pad="C"/>
+<wire x1="-23.615" y1="2.54" x2="-21.075" y2="5.08" width="0.8128" layer="16"/>
+<wire x1="-21.075" y1="5.08" x2="-15.621" y2="5.08" width="0.8128" layer="16"/>
+<wire x1="-15.621" y1="5.08" x2="-13.2878" y2="2.7468" width="0.8128" layer="16"/>
+<wire x1="-13.2878" y1="2.7468" x2="-13.2878" y2="1.43184375" width="0.8128" layer="16"/>
+<wire x1="-11.125" y1="-0.73095625" x2="-11.125" y2="-2.2225" width="0.8128" layer="16"/>
+<wire x1="-13.2878" y1="1.43184375" x2="-11.125" y2="-0.73095625" width="0.8128" layer="16"/>
+</signal>
+<signal name="N$11">
+<contactref element="X2" pad="3"/>
+<contactref element="D2" pad="C"/>
+<wire x1="-2.225" y1="2.2225" x2="-2.225" y2="5.647" width="0.8128" layer="1"/>
+<wire x1="-2.225" y1="5.647" x2="-3.302" y2="6.724" width="0.8128" layer="1"/>
 </signal>
 </signals>
