File: Platine_2.brd (EAGLE design)
At the start: 88.9 x 101.6 mm, 21 parts, among them X2 DTF13-12PA

Commit message: update
Parts:
- BLINKER_LINKS, BLINKER_RECHTS: value Gelb -> 151054GS03000
- BREMSLEUCHTE, LICHT_LINKS, LICHT_RECHTS: value Rot -> 151054RS03000
- LADELEITUNG, NEBELSCHLUSSLEUCHTE, RUECKFAHRLEUCHTE, STROMVERSORGUNG: value Grün -> 151054GS03000

Commit message: blinker gelb !
Parts:
- BLINKER_LINKS, BLINKER_RECHTS: value 151054GS03000 -> 151054YS04500
Changed lines of the file:
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@@
 <attribute name="VALUE" x="-18" y="-35.5" size="1.778" layer="27"/>
 </element>
-<element name="BLINKER_LINKS" library="Wurth_LEDs_WL-TMRW" library_urn="urn:adsk.eagle:library:19063499" package="WL-TMRW_5MM" package3d_urn="urn:adsk.eagle:package:19063507/3" value="151054GS03000" x="-25.4" y="38.1" smashed="yes" rot="R90">
-<attribute name="CHIP-TECHNOLOGY" value="InGaN" x="-25.4" y="38.1" size="1.778" layer="27" rot="R90" display="off"/>
-<attribute name="DATASHEET-URL" value="https://www.we-online.com/redexpert/spec/151054GS03000?ae" x="-25.4" y="38.1" size="1.778" layer="27" rot="R90" display="off"/>
-<attribute name="DOMINANT-WAVELENGTH" value="522nm" x="-25.4" y="38.1" size="1.778" layer="27" rot="R90" display="off"/>
-<attribute name="EMITTING-COLOR" value="Green" x="-25.4" y="38.1" size="1.778" layer="27" rot="R90" display="off"/>
-<attribute name="FORWARD-VOLTAGE" value="3.4V" x="-25.4" y="38.1" size="1.778" layer="27" rot="R90" display="off"/>
-<attribute name="LUMINOUS-INTENSITY" value="10000mcd" x="-25.4" y="38.1" size="1.778" layer="27" rot="R90" display="off"/>
+<element name="BLINKER_LINKS" library="Wurth_LEDs_WL-TMRW" library_urn="urn:adsk.eagle:library:19063499" package="WL-TMRW_5MM" package3d_urn="urn:adsk.eagle:package:19063507/3" value="151054YS04500" x="-25.4" y="38.1" smashed="yes" rot="R90">
+<attribute name="CHIP-TECHNOLOGY" value="AlInGaP" x="-25.4" y="38.1" size="1.778" layer="27" rot="R90" display="off"/>
+<attribute name="DATASHEET-URL" value="https://www.we-online.com/redexpert/spec/151054YS04500?ae" x="-25.4" y="38.1" size="1.778" layer="27" rot="R90" display="off"/>
+<attribute name="DOMINANT-WAVELENGTH" value="590nm" x="-25.4" y="38.1" size="1.778" layer="27" rot="R90" display="off"/>
+<attribute name="EMITTING-COLOR" value="Yellow" x="-25.4" y="38.1" size="1.778" layer="27" rot="R90" display="off"/>
+<attribute name="FORWARD-VOLTAGE" value="2.1V" x="-25.4" y="38.1" size="1.778" layer="27" rot="R90" display="off"/>
+<attribute name="LUMINOUS-INTENSITY" value="1500mcd" x="-25.4" y="38.1" size="1.778" layer="27" rot="R90" display="off"/>
 <attribute name="NAME" x="-25.4" y="41.91" size="0.8128" layer="25" align="bottom-center"/>
-<attribute name="PART-NUMBER" value="151054GS03000" x="-25.4" y="38.1" size="1.778" layer="27" rot="R90" display="off"/>
-<attribute name="PEAK-WAVELENGTH" value="515nm" x="-25.4" y="38.1" size="1.778" layer="27" rot="R90" display="off"/>
-<attribute name="VALUE" value="151054GS03000" x="-21.205" y="38.017" size="0.8128" layer="27" rot="R90" align="bottom-center"/>
-<attribute name="VIEWING-ANGLE" value="30°" x="-25.4" y="38.1" size="1.778" layer="27" rot="R90" display="off"/>
+<attribute name="PART-NUMBER" value="151054YS04500" x="-25.4" y="38.1" size="1.778" layer="27" rot="R90" display="off"/>
+<attribute name="PEAK-WAVELENGTH" value="592nm" x="-25.4" y="38.1" size="1.778" layer="27" rot="R90" display="off"/>
+<attribute name="VALUE" value="151054YS04500" x="-21.205" y="38.017" size="0.8128" layer="27" rot="R90" align="bottom-center"/>
+<attribute name="VIEWING-ANGLE" value="45°" x="-25.4" y="38.1" size="1.778" layer="27" rot="R90" display="off"/>
 </element>
-<element name="BLINKER_RECHTS" library="Wurth_LEDs_WL-TMRW" library_urn="urn:adsk.eagle:library:19063499" package="WL-TMRW_5MM" package3d_urn="urn:adsk.eagle:package:19063507/3" value="151054GS03000" x="25.4" y="38.1" smashed="yes" rot="R90">
-<attribute name="CHIP-TECHNOLOGY" value="InGaN" x="25.4" y="38.1" size="1.778" layer="27" rot="R90" display="off"/>
-<attribute name="DATASHEET-URL" value="https://www.we-online.com/redexpert/spec/151054GS03000?ae" x="25.4" y="38.1" size="1.778" layer="27" rot="R90" display="off"/>
-<attribute name="DOMINANT-WAVELENGTH" value="522nm" x="25.4" y="38.1" size="1.778" layer="27" rot="R90" display="off"/>
-<attribute name="EMITTING-COLOR" value="Green" x="25.4" y="38.1" size="1.778" layer="27" rot="R90" display="off"/>
-<attribute name="FORWARD-VOLTAGE" value="3.4V" x="25.4" y="38.1" size="1.778" layer="27" rot="R90" display="off"/>
-<attribute name="LUMINOUS-INTENSITY" value="10000mcd" x="25.4" y="38.1" size="1.778" layer="27" rot="R90" display="off"/>
+<element name="BLINKER_RECHTS" library="Wurth_LEDs_WL-TMRW" library_urn="urn:adsk.eagle:library:19063499" package="WL-TMRW_5MM" package3d_urn="urn:adsk.eagle:package:19063507/3" value="151054YS04500" x="25.4" y="38.1" smashed="yes" rot="R90">
+<attribute name="CHIP-TECHNOLOGY" value="AlInGaP" x="25.4" y="38.1" size="1.778" layer="27" rot="R90" display="off"/>
+<attribute name="DATASHEET-URL" value="https://www.we-online.com/redexpert/spec/151054YS04500?ae" x="25.4" y="38.1" size="1.778" layer="27" rot="R90" display="off"/>
+<attribute name="DOMINANT-WAVELENGTH" value="590nm" x="25.4" y="38.1" size="1.778" layer="27" rot="R90" display="off"/>
+<attribute name="EMITTING-COLOR" value="Yellow" x="25.4" y="38.1" size="1.778" layer="27" rot="R90" display="off"/>
+<attribute name="FORWARD-VOLTAGE" value="2.1V" x="25.4" y="38.1" size="1.778" layer="27" rot="R90" display="off"/>
+<attribute name="LUMINOUS-INTENSITY" value="1500mcd" x="25.4" y="38.1" size="1.778" layer="27" rot="R90" display="off"/>
 <attribute name="NAME" x="25.4" y="41.91" size="0.8128" layer="25" align="bottom-center"/>
-<attribute name="PART-NUMBER" value="151054GS03000" x="25.4" y="38.1" size="1.778" layer="27" rot="R90" display="off"/>
-<attribute name="PEAK-WAVELENGTH" value="515nm" x="25.4" y="38.1" size="1.778" layer="27" rot="R90" display="off"/>
-<attribute name="VALUE" value="151054GS03000" x="29.595" y="38.017" size="0.8128" layer="27" rot="R90" align="bottom-center"/>
-<attribute name="VIEWING-ANGLE" value="30°" x="25.4" y="38.1" size="1.778" layer="27" rot="R90" display="off"/>
+<attribute name="PART-NUMBER" value="151054YS04500" x="25.4" y="38.1" size="1.778" layer="27" rot="R90" display="off"/>
+<attribute name="PEAK-WAVELENGTH" value="592nm" x="25.4" y="38.1" size="1.778" layer="27" rot="R90" display="off"/>
+<attribute name="VALUE" value="151054YS04500" x="29.595" y="38.017" size="0.8128" layer="27" rot="R90" align="bottom-center"/>
+<attribute name="VIEWING-ANGLE" value="45°" x="25.4" y="38.1" size="1.778" layer="27" rot="R90" display="off"/>
 </element>
 <element name="R2" library="resistor" library_urn="urn:adsk.eagle:library:348" package="0204/7" package3d_urn="urn:adsk.eagle:package:23498/2" value="680" x="-31.75" y="35.56" smashed="yes" rot="R90">
