File: Platine_2_smd.brd (EAGLE design)
At the start: 88.9 x 101.6 mm, 21 parts, among them X2 DTF13-12PA

Commit message: REV
Parts:
- BLINKER_LINKS, BLINKER_RECHTS, LADELEITUNG, NEBELSCHLUSSLEUCHTE, RUECKFAHRLEUCHTE, STROMVERSORGUNG: device Wurth_LEDs_WL-SMRW:WL-SMRW_1206_DOME -> Wurth_LEDs_WL-SMRW:WL-SMRW_1206_DOME_REV
