File: Platine_2_smd.sch (EAGLE design)
At the start: 21 parts, among them X2 DTF13-12PA

Commit message: Updated Libraries !
Parts:
- BLINKER_LINKS, BLINKER_RECHTS: value Gelb -> 156120SS82500
- BREMSLEUCHTE, LICHT_LINKS, LICHT_RECHTS: value Rot -> 156120SS82500
- LADELEITUNG, NEBELSCHLUSSLEUCHTE, RUECKFAHRLEUCHTE, STROMVERSORGUNG: value Grün -> 156120SS82500
Changed lines of the file:
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@@
 </classes>
 <parts>
-<part name="X2" library="DEUTSCH-PCB" library_urn="urn:adsk.eagle:library:32238108" deviceset="DTF13-12PA" device="" package3d_urn="urn:adsk.eagle:package:32238112/2"/>
-<part name="BLINKER_LINKS" library="Wurth_LEDs_WL-SMRW" library_urn="urn:adsk.eagle:library:19040144" deviceset="WL-SMRW_1206_DOME" device="_REV" package3d_urn="urn:adsk.eagle:package:19040154/2" technology="_156120SS82500" value="Gelb"/>
-<part name="BLINKER_RECHTS" library="Wurth_LEDs_WL-SMRW" library_urn="urn:adsk.eagle:library:19040144" deviceset="WL-SMRW_1206_DOME" device="_REV" package3d_urn="urn:adsk.eagle:package:19040154/2" technology="_156120SS82500" value="Gelb"/>
+<part name="X2" library="DEUTSCH-PCB" library_urn="urn:adsk.eagle:library:32238108" deviceset="DTF13-12PA" device="" package3d_urn="urn:adsk.eagle:package:32238112/3"/>
+<part name="BLINKER_LINKS" library="Wurth_LEDs_WL-SMRW" library_urn="urn:adsk.eagle:library:19040144" deviceset="WL-SMRW_1206_DOME" device="_REV" package3d_urn="urn:adsk.eagle:package:19040154/3" technology="_156120SS82500" value="156120SS82500"/>
+<part name="BLINKER_RECHTS" library="Wurth_LEDs_WL-SMRW" library_urn="urn:adsk.eagle:library:19040144" deviceset="WL-SMRW_1206_DOME" device="_REV" package3d_urn="urn:adsk.eagle:package:19040154/3" technology="_156120SS82500" value="156120SS82500"/>
 <part name="R2" library="rcl" library_urn="urn:adsk.eagle:library:334" deviceset="R-EU_" device="R1206" package3d_urn="urn:adsk.eagle:package:23540/2" value="680"/>
 <part name="R1" library="rcl" library_urn="urn:adsk.eagle:library:334" deviceset="R-EU_" device="R1206" package3d_urn="urn:adsk.eagle:package:23540/2" value="680"/>
-<part name="LICHT_LINKS" library="Wurth_LEDs_WL-SMRW" library_urn="urn:adsk.eagle:library:19040144" deviceset="WL-SMRW_1206_DOME" device="_REV" package3d_urn="urn:adsk.eagle:package:19040154/2" technology="_156120SS82500" value="Rot"/>
-<part name="LICHT_RECHTS" library="Wurth_LEDs_WL-SMRW" library_urn="urn:adsk.eagle:library:19040144" deviceset="WL-SMRW_1206_DOME" device="_REV" package3d_urn="urn:adsk.eagle:package:19040154/2" technology="_156120SS82500" value="Rot"/>
-<part name="BREMSLEUCHTE" library="Wurth_LEDs_WL-SMRW" library_urn="urn:adsk.eagle:library:19040144" deviceset="WL-SMRW_1206_DOME" device="_REV" package3d_urn="urn:adsk.eagle:package:19040154/2" technology="_156120SS82500" value="Rot"/>
-<part name="NEBELSCHLUSSLEUCHTE" library="Wurth_LEDs_WL-SMRW" library_urn="urn:adsk.eagle:library:19040144" deviceset="WL-SMRW_1206_DOME" device="_REV" package3d_urn="urn:adsk.eagle:package:19040154/2" technology="_156120SS82500" value="Grün"/>
-<part name="STROMVERSORGUNG" library="Wurth_LEDs_WL-SMRW" library_urn="urn:adsk.eagle:library:19040144" deviceset="WL-SMRW_1206_DOME" device="_REV" package3d_urn="urn:adsk.eagle:package:19040154/2" technology="_156120SS82500" value="Grün"/>
-<part name="LADELEITUNG" library="Wurth_LEDs_WL-SMRW" library_urn="urn:adsk.eagle:library:19040144" deviceset="WL-SMRW_1206_DOME" device="_REV" package3d_urn="urn:adsk.eagle:package:19040154/2" technology="_156120SS82500" value="Grün"/>
+<part name="LICHT_LINKS" library="Wurth_LEDs_WL-SMRW" library_urn="urn:adsk.eagle:library:19040144" deviceset="WL-SMRW_1206_DOME" device="_REV" package3d_urn="urn:adsk.eagle:package:19040154/3" technology="_156120SS82500" value="156120SS82500"/>
+<part name="LICHT_RECHTS" library="Wurth_LEDs_WL-SMRW" library_urn="urn:adsk.eagle:library:19040144" deviceset="WL-SMRW_1206_DOME" device="_REV" package3d_urn="urn:adsk.eagle:package:19040154/3" technology="_156120SS82500" value="156120SS82500"/>
+<part name="BREMSLEUCHTE" library="Wurth_LEDs_WL-SMRW" library_urn="urn:adsk.eagle:library:19040144" deviceset="WL-SMRW_1206_DOME" device="_REV" package3d_urn="urn:adsk.eagle:package:19040154/3" technology="_156120SS82500" value="156120SS82500"/>
+<part name="NEBELSCHLUSSLEUCHTE" library="Wurth_LEDs_WL-SMRW" library_urn="urn:adsk.eagle:library:19040144" deviceset="WL-SMRW_1206_DOME" device="_REV" package3d_urn="urn:adsk.eagle:package:19040154/3" technology="_156120SS82500" value="156120SS82500"/>
+<part name="STROMVERSORGUNG" library="Wurth_LEDs_WL-SMRW" library_urn="urn:adsk.eagle:library:19040144" deviceset="WL-SMRW_1206_DOME" device="_REV" package3d_urn="urn:adsk.eagle:package:19040154/3" technology="_156120SS82500" value="156120SS82500"/>
+<part name="LADELEITUNG" library="Wurth_LEDs_WL-SMRW" library_urn="urn:adsk.eagle:library:19040144" deviceset="WL-SMRW_1206_DOME" device="_REV" package3d_urn="urn:adsk.eagle:package:19040154/3" technology="_156120SS82500" value="156120SS82500"/>
 <part name="R3" library="rcl" library_urn="urn:adsk.eagle:library:334" deviceset="R-EU_" device="R1206" package3d_urn="urn:adsk.eagle:package:23540/2" value="680"/>
 <part name="R4" library="rcl" library_urn="urn:adsk.eagle:library:334" deviceset="R-EU_" device="R1206" package3d_urn="urn:adsk.eagle:package:23540/2" value="680"/>
@@
 <part name="R7" library="rcl" library_urn="urn:adsk.eagle:library:334" deviceset="R-EU_" device="R1206" package3d_urn="urn:adsk.eagle:package:23540/2" value="680"/>
 <part name="R8" library="rcl" library_urn="urn:adsk.eagle:library:334" deviceset="R-EU_" device="R1206" package3d_urn="urn:adsk.eagle:package:23540/2" value="680"/>
-<part name="RUECKFAHRLEUCHTE" library="Wurth_LEDs_WL-SMRW" library_urn="urn:adsk.eagle:library:19040144" deviceset="WL-SMRW_1206_DOME" device="_REV" package3d_urn="urn:adsk.eagle:package:19040154/2" technology="_156120SS82500" value="Grün"/>
+<part name="RUECKFAHRLEUCHTE" library="Wurth_LEDs_WL-SMRW" library_urn="urn:adsk.eagle:library:19040144" deviceset="WL-SMRW_1206_DOME" device="_REV" package3d_urn="urn:adsk.eagle:package:19040154/3" technology="_156120SS82500" value="156120SS82500"/>
 <part name="R9" library="rcl" library_urn="urn:adsk.eagle:library:334" deviceset="R-EU_" device="R1206" package3d_urn="urn:adsk.eagle:package:23540/2" value="680"/>
 <part name="FRAME1" library="frames" library_urn="urn:adsk.eagle:library:229" deviceset="A4P-LOC" device=""/>

Commit message: Farben der LEDS
Parts:
- added D3: 156120VS82500, Wurth_LEDs_WL-SMRW:WL-SMRW_1206_DOME_156120VS82500_NOR
- BLINKER_LINKS, BLINKER_RECHTS: value 156120SS82500 -> 156120YS82500; device Wurth_LEDs_WL-SMRW:WL-SMRW_1206_DOME_156120SS82500_REV -> Wurth_LEDs_WL-SMRW:WL-SMRW_1206_DOME_156120YS82500_NOR
- LADELEITUNG, NEBELSCHLUSSLEUCHTE, RUECKFAHRLEUCHTE, STROMVERSORGUNG: value 156120SS82500 -> 156120VS82500; device Wurth_LEDs_WL-SMRW:WL-SMRW_1206_DOME_156120SS82500_REV -> Wurth_LEDs_WL-SMRW:WL-SMRW_1206_DOME_156120VS82500_NOR
Changed lines of the file:
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@@
 <parts>
 <part name="X2" library="DEUTSCH-PCB" library_urn="urn:adsk.eagle:library:32238108" deviceset="DTF13-12PA" device="" package3d_urn="urn:adsk.eagle:package:32238112/3"/>
-<part name="BLINKER_LINKS" library="Wurth_LEDs_WL-SMRW" library_urn="urn:adsk.eagle:library:19040144" deviceset="WL-SMRW_1206_DOME" device="_REV" package3d_urn="urn:adsk.eagle:package:19040154/3" technology="_156120SS82500" value="156120SS82500"/>
-<part name="BLINKER_RECHTS" library="Wurth_LEDs_WL-SMRW" library_urn="urn:adsk.eagle:library:19040144" deviceset="WL-SMRW_1206_DOME" device="_REV" package3d_urn="urn:adsk.eagle:package:19040154/3" technology="_156120SS82500" value="156120SS82500"/>
+<part name="BLINKER_LINKS" library="Wurth_LEDs_WL-SMRW" library_urn="urn:adsk.eagle:library:19040144" deviceset="WL-SMRW_1206_DOME" device="_NOR" package3d_urn="urn:adsk.eagle:package:19040155/3" technology="_156120YS82500" value="156120YS82500"/>
+<part name="BLINKER_RECHTS" library="Wurth_LEDs_WL-SMRW" library_urn="urn:adsk.eagle:library:19040144" deviceset="WL-SMRW_1206_DOME" device="_NOR" package3d_urn="urn:adsk.eagle:package:19040155/3" technology="_156120YS82500" value="156120YS82500"/>
 <part name="R2" library="rcl" library_urn="urn:adsk.eagle:library:334" deviceset="R-EU_" device="R1206" package3d_urn="urn:adsk.eagle:package:23540/2" value="680"/>
 <part name="R1" library="rcl" library_urn="urn:adsk.eagle:library:334" deviceset="R-EU_" device="R1206" package3d_urn="urn:adsk.eagle:package:23540/2" value="680"/>
@@
 <part name="LICHT_RECHTS" library="Wurth_LEDs_WL-SMRW" library_urn="urn:adsk.eagle:library:19040144" deviceset="WL-SMRW_1206_DOME" device="_REV" package3d_urn="urn:adsk.eagle:package:19040154/3" technology="_156120SS82500" value="156120SS82500"/>
 <part name="BREMSLEUCHTE" library="Wurth_LEDs_WL-SMRW" library_urn="urn:adsk.eagle:library:19040144" deviceset="WL-SMRW_1206_DOME" device="_REV" package3d_urn="urn:adsk.eagle:package:19040154/3" technology="_156120SS82500" value="156120SS82500"/>
-<part name="NEBELSCHLUSSLEUCHTE" library="Wurth_LEDs_WL-SMRW" library_urn="urn:adsk.eagle:library:19040144" deviceset="WL-SMRW_1206_DOME" device="_REV" package3d_urn="urn:adsk.eagle:package:19040154/3" technology="_156120SS82500" value="156120SS82500"/>
-<part name="STROMVERSORGUNG" library="Wurth_LEDs_WL-SMRW" library_urn="urn:adsk.eagle:library:19040144" deviceset="WL-SMRW_1206_DOME" device="_REV" package3d_urn="urn:adsk.eagle:package:19040154/3" technology="_156120SS82500" value="156120SS82500"/>
-<part name="LADELEITUNG" library="Wurth_LEDs_WL-SMRW" library_urn="urn:adsk.eagle:library:19040144" deviceset="WL-SMRW_1206_DOME" device="_REV" package3d_urn="urn:adsk.eagle:package:19040154/3" technology="_156120SS82500" value="156120SS82500"/>
+<part name="NEBELSCHLUSSLEUCHTE" library="Wurth_LEDs_WL-SMRW" library_urn="urn:adsk.eagle:library:19040144" deviceset="WL-SMRW_1206_DOME" device="_NOR" package3d_urn="urn:adsk.eagle:package:19040155/3" technology="_156120VS82500" value="156120VS82500"/>
+<part name="STROMVERSORGUNG" library="Wurth_LEDs_WL-SMRW" library_urn="urn:adsk.eagle:library:19040144" deviceset="WL-SMRW_1206_DOME" device="_NOR" package3d_urn="urn:adsk.eagle:package:19040155/3" technology="_156120VS82500" value="156120VS82500"/>
+<part name="LADELEITUNG" library="Wurth_LEDs_WL-SMRW" library_urn="urn:adsk.eagle:library:19040144" deviceset="WL-SMRW_1206_DOME" device="_NOR" package3d_urn="urn:adsk.eagle:package:19040155/3" technology="_156120VS82500" value="156120VS82500"/>
 <part name="R3" library="rcl" library_urn="urn:adsk.eagle:library:334" deviceset="R-EU_" device="R1206" package3d_urn="urn:adsk.eagle:package:23540/2" value="680"/>
 <part name="R4" library="rcl" library_urn="urn:adsk.eagle:library:334" deviceset="R-EU_" device="R1206" package3d_urn="urn:adsk.eagle:package:23540/2" value="680"/>
@@
 <part name="R7" library="rcl" library_urn="urn:adsk.eagle:library:334" deviceset="R-EU_" device="R1206" package3d_urn="urn:adsk.eagle:package:23540/2" value="680"/>
 <part name="R8" library="rcl" library_urn="urn:adsk.eagle:library:334" deviceset="R-EU_" device="R1206" package3d_urn="urn:adsk.eagle:package:23540/2" value="680"/>
-<part name="RUECKFAHRLEUCHTE" library="Wurth_LEDs_WL-SMRW" library_urn="urn:adsk.eagle:library:19040144" deviceset="WL-SMRW_1206_DOME" device="_REV" package3d_urn="urn:adsk.eagle:package:19040154/3" technology="_156120SS82500" value="156120SS82500"/>
+<part name="RUECKFAHRLEUCHTE" library="Wurth_LEDs_WL-SMRW" library_urn="urn:adsk.eagle:library:19040144" deviceset="WL-SMRW_1206_DOME" device="_NOR" package3d_urn="urn:adsk.eagle:package:19040155/3" technology="_156120VS82500" value="156120VS82500"/>
 <part name="R9" library="rcl" library_urn="urn:adsk.eagle:library:334" deviceset="R-EU_" device="R1206" package3d_urn="urn:adsk.eagle:package:23540/2" value="680"/>
 <part name="FRAME1" library="frames" library_urn="urn:adsk.eagle:library:229" deviceset="A4P-LOC" device=""/>
@@
 <part name="D1" library="diode" library_urn="urn:adsk.eagle:library:210" deviceset="MBRS130LT3" device="" package3d_urn="urn:adsk.eagle:package:43404/2"/>
 <part name="D2" library="diode" library_urn="urn:adsk.eagle:library:210" deviceset="MBRS130LT3" device="" package3d_urn="urn:adsk.eagle:package:43404/2"/>
+<part name="D3" library="Wurth_LEDs_WL-SMRW" library_urn="urn:adsk.eagle:library:19040144" deviceset="WL-SMRW_1206_DOME" device="_NOR" package3d_urn="urn:adsk.eagle:package:19040155/3" technology="_156120VS82500" value="156120VS82500"/>
 </parts>
 <sheets>
@@
 <attribute name="VALUE" x="145.542" y="85.09" size="1.778" layer="96" rot="R90"/>
 </instance>
+<instance part="D3" gate="G$1" x="20.32" y="109.22" smashed="yes">
+<attribute name="NAME" x="20.872" y="113.592" size="1.27" layer="95" align="bottom-center"/>
+<attribute name="VALUE" x="20.932" y="105.492" size="1.27" layer="96" align="bottom-center"/>
+</instance>
 </instances>

Commit message: ..
Parts:
- removed D3: 156120VS82500, Wurth_LEDs_WL-SMRW:WL-SMRW_1206_DOME_156120VS82500_NOR
Changed lines of the file:
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@@
 <part name="D1" library="diode" library_urn="urn:adsk.eagle:library:210" deviceset="MBRS130LT3" device="" package3d_urn="urn:adsk.eagle:package:43404/2"/>
 <part name="D2" library="diode" library_urn="urn:adsk.eagle:library:210" deviceset="MBRS130LT3" device="" package3d_urn="urn:adsk.eagle:package:43404/2"/>
-<part name="D3" library="Wurth_LEDs_WL-SMRW" library_urn="urn:adsk.eagle:library:19040144" deviceset="WL-SMRW_1206_DOME" device="_NOR" package3d_urn="urn:adsk.eagle:package:19040155/3" technology="_156120VS82500" value="156120VS82500"/>
 </parts>
 <sheets>
@@
 <attribute name="VALUE" x="145.542" y="85.09" size="1.778" layer="96" rot="R90"/>
 </instance>
-<instance part="D3" gate="G$1" x="20.32" y="109.22" smashed="yes">
-<attribute name="NAME" x="20.872" y="113.592" size="1.27" layer="95" align="bottom-center"/>
-<attribute name="VALUE" x="20.932" y="105.492" size="1.27" layer="96" align="bottom-center"/>
-</instance>
 </instances>

Commit message: REV
Parts:
- BLINKER_LINKS, BLINKER_RECHTS: device Wurth_LEDs_WL-SMRW:WL-SMRW_1206_DOME_156120YS82500_NOR -> Wurth_LEDs_WL-SMRW:WL-SMRW_1206_DOME_156120YS82500_REV
- LADELEITUNG, NEBELSCHLUSSLEUCHTE, RUECKFAHRLEUCHTE, STROMVERSORGUNG: device Wurth_LEDs_WL-SMRW:WL-SMRW_1206_DOME_156120VS82500_NOR -> Wurth_LEDs_WL-SMRW:WL-SMRW_1206_DOME_156120SS82500_REV
Changed lines of the file:
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@@
 <parts>
 <part name="X2" library="DEUTSCH-PCB" library_urn="urn:adsk.eagle:library:32238108" deviceset="DTF13-12PA" device="" package3d_urn="urn:adsk.eagle:package:32238112/3"/>
-<part name="BLINKER_LINKS" library="Wurth_LEDs_WL-SMRW" library_urn="urn:adsk.eagle:library:19040144" deviceset="WL-SMRW_1206_DOME" device="_NOR" package3d_urn="urn:adsk.eagle:package:19040155/3" technology="_156120YS82500" value="156120YS82500"/>
-<part name="BLINKER_RECHTS" library="Wurth_LEDs_WL-SMRW" library_urn="urn:adsk.eagle:library:19040144" deviceset="WL-SMRW_1206_DOME" device="_NOR" package3d_urn="urn:adsk.eagle:package:19040155/3" technology="_156120YS82500" value="156120YS82500"/>
+<part name="BLINKER_LINKS" library="Wurth_LEDs_WL-SMRW" library_urn="urn:adsk.eagle:library:19040144" deviceset="WL-SMRW_1206_DOME" device="_REV" package3d_urn="urn:adsk.eagle:package:19040154/3" technology="_156120YS82500" value="156120YS82500"/>
+<part name="BLINKER_RECHTS" library="Wurth_LEDs_WL-SMRW" library_urn="urn:adsk.eagle:library:19040144" deviceset="WL-SMRW_1206_DOME" device="_REV" package3d_urn="urn:adsk.eagle:package:19040154/3" technology="_156120YS82500" value="156120YS82500"/>
 <part name="R2" library="rcl" library_urn="urn:adsk.eagle:library:334" deviceset="R-EU_" device="R1206" package3d_urn="urn:adsk.eagle:package:23540/2" value="680"/>
 <part name="R1" library="rcl" library_urn="urn:adsk.eagle:library:334" deviceset="R-EU_" device="R1206" package3d_urn="urn:adsk.eagle:package:23540/2" value="680"/>
@@
 <part name="LICHT_RECHTS" library="Wurth_LEDs_WL-SMRW" library_urn="urn:adsk.eagle:library:19040144" deviceset="WL-SMRW_1206_DOME" device="_REV" package3d_urn="urn:adsk.eagle:package:19040154/3" technology="_156120SS82500" value="156120SS82500"/>
 <part name="BREMSLEUCHTE" library="Wurth_LEDs_WL-SMRW" library_urn="urn:adsk.eagle:library:19040144" deviceset="WL-SMRW_1206_DOME" device="_REV" package3d_urn="urn:adsk.eagle:package:19040154/3" technology="_156120SS82500" value="156120SS82500"/>
-<part name="NEBELSCHLUSSLEUCHTE" library="Wurth_LEDs_WL-SMRW" library_urn="urn:adsk.eagle:library:19040144" deviceset="WL-SMRW_1206_DOME" device="_NOR" package3d_urn="urn:adsk.eagle:package:19040155/3" technology="_156120VS82500" value="156120VS82500"/>
-<part name="STROMVERSORGUNG" library="Wurth_LEDs_WL-SMRW" library_urn="urn:adsk.eagle:library:19040144" deviceset="WL-SMRW_1206_DOME" device="_NOR" package3d_urn="urn:adsk.eagle:package:19040155/3" technology="_156120VS82500" value="156120VS82500"/>
-<part name="LADELEITUNG" library="Wurth_LEDs_WL-SMRW" library_urn="urn:adsk.eagle:library:19040144" deviceset="WL-SMRW_1206_DOME" device="_NOR" package3d_urn="urn:adsk.eagle:package:19040155/3" technology="_156120VS82500" value="156120VS82500"/>
+<part name="NEBELSCHLUSSLEUCHTE" library="Wurth_LEDs_WL-SMRW" library_urn="urn:adsk.eagle:library:19040144" deviceset="WL-SMRW_1206_DOME" device="_REV" package3d_urn="urn:adsk.eagle:package:19040154/3" technology="_156120SS82500" value="156120VS82500"/>
+<part name="STROMVERSORGUNG" library="Wurth_LEDs_WL-SMRW" library_urn="urn:adsk.eagle:library:19040144" deviceset="WL-SMRW_1206_DOME" device="_REV" package3d_urn="urn:adsk.eagle:package:19040154/3" technology="_156120SS82500" value="156120VS82500"/>
+<part name="LADELEITUNG" library="Wurth_LEDs_WL-SMRW" library_urn="urn:adsk.eagle:library:19040144" deviceset="WL-SMRW_1206_DOME" device="_REV" package3d_urn="urn:adsk.eagle:package:19040154/3" technology="_156120SS82500" value="156120VS82500"/>
 <part name="R3" library="rcl" library_urn="urn:adsk.eagle:library:334" deviceset="R-EU_" device="R1206" package3d_urn="urn:adsk.eagle:package:23540/2" value="680"/>
 <part name="R4" library="rcl" library_urn="urn:adsk.eagle:library:334" deviceset="R-EU_" device="R1206" package3d_urn="urn:adsk.eagle:package:23540/2" value="680"/>
@@
 <part name="R7" library="rcl" library_urn="urn:adsk.eagle:library:334" deviceset="R-EU_" device="R1206" package3d_urn="urn:adsk.eagle:package:23540/2" value="680"/>
 <part name="R8" library="rcl" library_urn="urn:adsk.eagle:library:334" deviceset="R-EU_" device="R1206" package3d_urn="urn:adsk.eagle:package:23540/2" value="680"/>
-<part name="RUECKFAHRLEUCHTE" library="Wurth_LEDs_WL-SMRW" library_urn="urn:adsk.eagle:library:19040144" deviceset="WL-SMRW_1206_DOME" device="_NOR" package3d_urn="urn:adsk.eagle:package:19040155/3" technology="_156120VS82500" value="156120VS82500"/>
+<part name="RUECKFAHRLEUCHTE" library="Wurth_LEDs_WL-SMRW" library_urn="urn:adsk.eagle:library:19040144" deviceset="WL-SMRW_1206_DOME" device="_REV" package3d_urn="urn:adsk.eagle:package:19040154/3" technology="_156120SS82500" value="156120VS82500"/>
 <part name="R9" library="rcl" library_urn="urn:adsk.eagle:library:334" deviceset="R-EU_" device="R1206" package3d_urn="urn:adsk.eagle:package:23540/2" value="680"/>
 <part name="FRAME1" library="frames" library_urn="urn:adsk.eagle:library:229" deviceset="A4P-LOC" device=""/>
